File: src/frog.kicad_pcb (KiCad board)
At the start: 2 copper layers, 80.5 x 45.9 mm, 10 parts, among them SW1 SW_Push

Commit message: .
Parts:
- added G***: LOGO, LOGO, F.Cu at (109.0, 113.5)
- added G***: LOGO, LOGO, F.Cu at (175.4, 113.7)
- added G***: LOGO, LOGO, B.Cu at (166.9, 109.9)
- added G***: LOGO, LOGO, B.Cu at (142.1, 110.0)
- added G***: LOGO, LOGO, B.Cu at (116.6, 108.1)
Routing:
- net Net-(BT1--): vias 3 -> 2
- net (no net): vias 0 -> 1
